Commit message: Added velocity ramp. Fixed issue with angular velocity on the tcp-server. Added launch files for bringing up the real robot.

File: src/mar_description/urdf/mar_model.urdf (robot description, URDF)
Before this commit: robot MAR, 12 links, 11 joints
Links:
- removed link camera_depth_frame
- removed link camera_link
- removed link sim_camera_depth_frame
- added link openni_depth_optical_frame, mass 0.0001
- added link openni_link, mass 0.0001; visual box size=0.064 0.121 0.0381
- added link openni_rgb_optical_frame, mass 0.0001
- link drive_compartment: mass 15 -> 1.2
- link laser: mass 0.2 -> 0.0001
- link rear_compartment: mass 1 -> 20
Joints:
- removed joint sim_camera_depth_joint
- added joint camera_rgb_joint: type fixed, parent openni_link, child openni_rgb_optical_frame, origin xyz=0 -0.01 0 rpy=-1.57 0 -1.57
- joint camera_depth_joint: child camera_depth_frame -> openni_depth_optical_frame; origin xyz=0 0.028 0 rpy=0 0 0 -> xyz=0 0.02 0 rpy=-1.57 0 -1.57; parent camera_link -> openni_link
- joint camera_frame_joint: child camera_link -> openni_link; origin xyz=0.36 0 0.13 -> xyz=0.38 0 0.13
